File: BQPowerSupply.sch (KiCad schematic (older format))
At the start: 34 parts

Commit message: Rev 2 without voltage monitor, with SOT23-5 for LDO
Parts:
- removed Good,OutSw,RegSw1: Conn_01x03, Connector_PinHeader_2.54mm:PinHeader_1x03_P2.54mm_Vertical, symbol Connector_Generic:Conn_01x03
- removed LDO1: TPS7A02-4X2SON, myFootprints:DQN, symbol BQPowerSupply-rescue:TPS7A02-4X2SON-mySchemSym
- removed VOutSw1, VregSw1: Conn_01x02, Connector_PinHeader_2.54mm:PinHeader_1x02_P2.54mm_Vertical, symbol Connector_Generic:Conn_01x02
- removed Vmon1: TPS3839-3.1V, Package_TO_SOT_SMD:SOT-23, symbol BQPowerSupply-rescue:TPS3839-SOT-23-mySchemSym
- added JVOutSw1, JVRegSw1: Conn_01x03, Connector_PinHeader_2.54mm:PinHeader_1x03_P2.54mm_Vertical, symbol Connector_Generic:Conn_01x03
- added LDO1: TPS7A02_3.6, Package_TO_SOT_SMD:SOT-23-5, symbol Regulator_Linear:TPS7A05285PDBV
- ROK2: value 5.36M -> 4,42M
- ROK3: value 1M -> 0.510M
Connections:
- net GND: now also JVOutSw1.2 (Pin_2), JVRegSw1.2 (Pin_2), LDO1.2 (GND)
- net VBatOK: now also LDO1.3 (EN)
- net VOut: now also LDO1.1 (IN)
- net VOutSw: now also JVOutSw1.1 (Pin_1)
- net VOutSwEn: now also JVOutSw1.3 (Pin_3)
- net VRegSwEn: now also JVRegSw1.3 (Pin_3)
- net Vreg: now also LDO1.5 (OUT)
- net VregSw: now also JVRegSw1.1 (Pin_1)
Other:
- note added: "2"
- note added: "Solar cell in"
- note added: "Super capacitor storage"
- note added: "VBatOk rising 2.1V\nfalling 2.0V"
- note removed: "Logic signals"
- note removed: "VBatOk rising 2.4V\nfalling 2.2V"
- moved on the sheet: Super1
Changed lines of the file:
@@
 Comment4 ""
 $EndDescr
-Text Notes 7250 6800 0    60   ~ 0
+Text Notes 7150 6950 0    60   ~ 0
 TI BQ harvest solar, store super capacitor, regulate and switch power supply
 $Comp
@@
 P 3400 5100
 F 0 "ROK2" H 3600 5000 50  0000 C CNN
-F 1 "5.36M" H 3600 5100 50  0000 C CNN
+F 1 "4,42M" H 3600 5100 50  0000 C CNN
 F 2 "Resistor_SMD:R_0603_1608Metric" V 3330 5100 50  0001 C CNN
 F 3 "" H 3400 5100 50  0000 C CNN
@@
 VOvervolt 5.5V
 Text Notes 3200 6050 0    60   ~ 0
-VBatOk rising 2.4V\nfalling 2.2V
+VBatOk rising 2.1V\nfalling 2.0V
 $Comp
 L Device:R ROK3
@@
 P 3400 4800
 F 0 "ROK3" H 3600 4700 50  0000 C CNN
-F 1 "1M" H 3600 4800 50  0000 C CNN
+F 1 "0.510M" H 3600 4800 50  0000 C CNN
 F 2 "Resistor_SMD:R_0603_1608Metric" V 3330 4800 50  0001 C CNN
 F 3 "" H 3400 4800 50  0000 C CNN
@@
 $EndComp
 $Comp
-L Connector_Generic:Conn_01x02 VOutSw1
-U 1 1 5E95332C
-P 10350 3300
-F 0 "VOutSw1" H 10430 3292 50  0000 L CNN
-F 1 "Conn_01x02" H 10430 3201 50  0000 L CNN
-F 2 "Connector_PinHeader_2.54mm:PinHeader_1x02_P2.54mm_Vertical" H 10350 3300 50  0001 C CNN
-F 3 "~" H 10350 3300 50  0001 C CNN
-F 4 "stock" H 10350 3300 50  0001 C CNN "SourcePartNo"
-	1    10350 3300
-	1    0    0    -1
-$EndComp
-$Comp
-L Connector_Generic:Conn_01x02 VregSw1
-U 1 1 5E953AB6
-P 10400 5300
-F 0 "VregSw1" H 10480 5292 50  0000 L CNN
-F 1 "Conn_01x02" H 10480 5201 50  0000 L CNN
-F 2 "Connector_PinHeader_2.54mm:PinHeader_1x02_P2.54mm_Vertical" H 10400 5300 50  0001 C CNN
-F 3 "~" H 10400 5300 50  0001 C CNN
-	1    10400 5300
-	1    0    0    -1
-$EndComp
-$Comp
 L power:GND #PWR014
 U 1 1 5E95424E
@@
 L power:GND #PWR023
 U 1 1 5E955DB2
-P 10200 5400
-F 0 "#PWR023" H 10200 5150 50  0001 C CNN
-F 1 "GND" V 10200 5150 50  0000 C CNN
-F 2 "" H 10200 5400 50  0000 C CNN
-F 3 "" H 10200 5400 50  0000 C CNN
-	1    10200 5400
+P 10400 5350
+F 0 "#PWR023" H 10400 5100 50  0001 C CNN
+F 1 "GND" V 10400 5100 50  0000 C CNN
+F 2 "" H 10400 5350 50  0000 C CNN
+F 3 "" H 10400 5350 50  0000 C CNN
+	1    10400 5350
 	0    1    1    0
 $EndComp
 Text GLabel 3150 3450 2    60   Input ~ 0
 VOut
-$Comp
-L BQPowerSupply-rescue:TPS7A02-4X2SON-mySchemSym LDO1
-U 1 1 5E928A83
-P 8850 4400
-F 0 "LDO1" H 8850 4742 50  0000 C CNN
-F 1 "TPS7A02-4X2SON" H 8850 4651 50  0000 C CNN
-F 2 "myFootprints:DQN" H 8850 4725 50  0001 C CIN
-F 3 "http://www.ti.com/lit/ds/symlink/tps7a02.pdf" H 8850 4450 50  0001 C CNN
-F 4 "296-TPS7A0222PDQNRCT-ND " H 8850 4400 50  0001 C CNN "SourcePartNo"
-	1    8850 4400
-	1    0    0    -1
-$EndComp
-Text GLabel 9150 4400 2    60   Input ~ 0
+Text GLabel 8500 4100 0    60   Input ~ 0
 VOut
-Text GLabel 9150 4500 2    60   Input ~ 0
+Text GLabel 8500 4200 0    60   Input ~ 0
 VBatOK
-$Comp
-L power:GND #PWR013
-U 1 1 5E929BA4
-P 9150 4300
-F 0 "#PWR013" H 9150 4050 50  0001 C CNN
-F 1 "GND" V 9150 4050 50  0000 C CNN
-F 2 "" H 9150 4300 50  0000 C CNN
-F 3 "" H 9150 4300 50  0000 C CNN
-	1    9150 4300
-	0    -1   -1   0
-$EndComp
 $Comp
 L power:GND #PWR012
 U 1 1 5E92A674
-P 8550 4500
-F 0 "#PWR012" H 8550 4250 50  0001 C CNN
-F 1 "GND" V 8550 4250 50  0000 C CNN
-F 2 "" H 8550 4500 50  0000 C CNN
-F 3 "" H 8550 4500 50  0000 C CNN
-	1    8550 4500
-	0    1    1    0
+P 8800 4500
+F 0 "#PWR012" H 8800 4250 50  0001 C CNN
+F 1 "GND" V 8800 4250 50  0000 C CNN
+F 2 "" H 8800 4500 50  0000 C CNN
+F 3 "" H 8800 4500 50  0000 C CNN
+	1    8800 4500
+	1    0    0    -1
 $EndComp
 Text GLabel 10150 2600 0    60   Input ~ 0
@@
 Text GLabel 8450 5250 0    60   Input ~ 0
 VregSw
-Text GLabel 10200 5300 0    60   Input ~ 0
+Text GLabel 10400 5250 0    60   Input ~ 0
 VregSw
-$Comp
-L BQPowerSupply-rescue:TPS3839-SOT-23-mySchemSym Vmon1
-U 1 1 5E938070
-P 8800 1800
-F 0 "Vmon1" H 8800 1887 60  0000 C CNN
-F 1 "TPS3839-3.1V" H 8800 1781 60  0000 C CNN
-F 2 "Package_TO_SOT_SMD:SOT-23" H 8800 1800 60  0001 C CNN
-F 3 "" H 8800 1800 60  0000 C CNN
-F 4 "296-35470-1-ND" H 8800 1800 50  0001 C CNN "SourcePartNo"
-	1    8800 1800
-	1    0    0    -1
-$EndComp
-Text GLabel 9250 2050 2    60   Input ~ 0
-VOut
-$Comp
-L power:GND #PWR010
-U 1 1 5E93A244
-P 8350 2000
-F 0 "#PWR010" H 8350 1750 50  0001 C CNN
-F 1 "GND" V 8350 1750 50  0000 C CNN
-F 2 "" H 8350 2000 50  0000 C CNN
-F 3 "" H 8350 2000 50  0000 C CNN
-	1    8350 2000
-	0    1    1    0
-$EndComp
-Text GLabel 8350 2150 0    60   Input ~ 0
-VOutGood
-Text GLabel 5100 7200 0    60   Output ~ 0
+Text GLabel 10150 3500 0    60   Output ~ 0
 VOutSwEn
 Text GLabel 9300 5250 2    60   Input ~ 0
 VRegSwEn
-Text GLabel 5100 7300 0    60   Output ~ 0
+Text GLabel 10400 5450 0    60   Output ~ 0
 VRegSwEn
-$Comp
-L Connector_Generic:Conn_01x03 Good,OutSw,RegSw1
-U 1 1 5E93C4D0
-P 5300 7200
-F 0 "Good,OutSw,RegSw1" H 5380 7242 50  0000 L CNN
-F 1 "Conn_01x03" H 5380 7151 50  0000 L CNN
-F 2 "Connector_PinHeader_2.54mm:PinHeader_1x03_P2.54mm_Vertical" H 5300 7200 50  0001 C CNN
-F 3 "~" H 5300 7200 50  0001 C CNN
-F 4 "stock" H 5300 7200 50  0001 C CNN "SourcePartNo"
-	1    5300 7200
-	1    0    0    -1
-$EndComp
-Text Notes 10300 2200 0    60   ~ 0
+Text Notes 9850 2200 0    60   ~ 0
 Power rails out
-Text Notes 4600 6650 0    60   ~ 0
-Logic signals
 $Comp
 L Device:C 1u1
@@
 	1    0    0    -1
 $EndComp
-Text GLabel 5100 7100 0    60   Input ~ 0
-VOutGood
 $Comp
 L power:GND #PWR0102
@@
 	-1   0    0    1
 $EndComp
-Text GLabel 4900 3250 0    60   Input ~ 0
+Text GLabel 4750 3750 0    60   Input ~ 0
 VOut
 $Comp
 L Connector_Generic:Conn_01x02 Super1
 U 1 1 5E94BEC9
-P 5100 3250
-F 0 "Super1" H 5018 2925 50  0000 C CNN
-F 1 "Conn_01x02" H 5018 3016 50  0000 C CNN
-F 2 "Connector_PinHeader_2.54mm:PinHeader_1x02_P2.54mm_Vertical" H 5100 3250 50  0001 C CNN
-F 3 "~" H 5100 3250 50  0001 C CNN
-	1    5100 3250
+P 4950 3750
+F 0 "Super1" H 4868 3425 50  0000 C CNN
+F 1 "Conn_01x02" H 4868 3516 50  0000 C CNN
+F 2 "Connector_PinHeader_2.54mm:PinHeader_1x02_P2.54mm_Vertical" H 4950 3750 50  0001 C CNN
+F 3 "~" H 4950 3750 50  0001 C CNN
+	1    4950 3750
 	1    0    0    -1
 $EndComp
@@
 L power:GND #PWR0103
 U 1 1 5E93BB4E
-P 4900 3350
-F 0 "#PWR0103" H 4900 3100 50  0001 C CNN
-F 1 "GND" V 4900 3150 50  0000 C CNN
-F 2 "" H 4900 3350 50  0000 C CNN
-F 3 "" H 4900 3350 50  0000 C CNN
-	1    4900 3350
+P 4750 3850
+F 0 "#PWR0103" H 4750 3600 50  0001 C CNN
+F 1 "GND" V 4750 3650 50  0000 C CNN
+F 2 "" H 4750 3850 50  0000 C CNN
+F 3 "" H 4750 3850 50  0000 C CNN
+	1    4750 3850
 	0    1    1    0
 $EndComp
@@
 	1    0    0    -1
 $EndComp
-Text GLabel 8550 4300 0    60   Input ~ 0
+Text GLabel 9100 4100 2    60   Input ~ 0
 Vreg
 Text Notes 5600 5950 0    60   ~ 0
 Note two filter caps on VReg can be combined if close together.
+Text Notes 4300 4250 0    60   ~ 0
+Super capacitor storage
+Text Notes 1000 700  0    60   ~ 0
+Solar cell in
+$Comp
+L Connector_Generic:Conn_01x03 JVOutSw1
+U 1 1 6250C90E
+P 10350 3400
+F 0 "JVOutSw1" H 10430 3442 50  0000 L CNN
+F 1 "Conn_01x03" H 10430 3351 50  0000 L CNN
+F 2 "Connector_PinHeader_2.54mm:PinHeader_1x03_P2.54mm_Vertical" H 10350 3400 50  0001 C CNN
+F 3 "~" H 10350 3400 50  0001 C CNN
+	1    10350 3400
+	1    0    0    -1
+$EndComp
+$Comp
+L Connector_Generic:Conn_01x03 JVRegSw1
+U 1 1 6250D938
+P 10600 5350
+F 0 "JVRegSw1" H 10680 5392 50  0000 L CNN
+F 1 "Conn_01x03" H 10680 5301 50  0000 L CNN
+F 2 "Connector_PinHeader_2.54mm:PinHeader_1x03_P2.54mm_Vertical" H 10600 5350 50  0001 C CNN
+F 3 "~" H 10600 5350 50  0001 C CNN
+	1    10600 5350
+	1    0    0    -1
+$EndComp
+Text Notes 10650 7650 0    60   ~ 0
+2
+$Comp
+L Regulator_Linear:TPS7A05285PDBV LDO1
+U 1 1 62518C58
+P 8800 4200
+F 0 "LDO1" H 8800 4567 50  0000 C CNN
+F 1 "TPS7A02_3.6" H 8800 4476 50  0000 C CNN
+F 2 "Package_TO_SOT_SMD:SOT-23-5" H 8800 4550 50  0001 C CNN
+F 3 "https://www.ti.com/lit/ds/symlink/tps7a05.pdf" H 8800 4700 50  0001 C CNN
+	1    8800 4200
+	1    0    0    -1
+$EndComp
 $EndSCHEMATC
